Commit message: added prefix property & argument

File: mrs_robot_launcher/urdf/X3/robot.urdf.xacro (robot description, xacro)
@@ -1,4 +1,6 @@
 <?xml version='1.0'?>
-<robot name = 'robot.urdf' xmlns:xacro = 'http://www.ros.org/wiki/xacro'>
+<robot name = '${robot.urdf}' xmlns:xacro = 'http://www.ros.org/wiki/xacro'>
+    <xacro:arg name = 'robot_name' default = 'robot1'/>
+    <xacro:property name = 'robot_name' value = '${arg robot_name}'/>
     <!-- include files -->
     <xacro:include filename = 'robot_body.xacro'/>

Commit message: added arguments on launch and properties based on arguments. for whatever reason, the properties are NOT global. need to fix

File: mrs_robot_launcher/urdf/X3/robot.urdf.xacro (robot description, xacro)
@@ -1,9 +1,9 @@
 <?xml version='1.0'?>
-<robot name = '${robot_name}.urdf' xmlns:xacro = 'http://www.ros.org/wiki/xacro'>
+<robot name = 'robot' xmlns:xacro = 'http://www.ros.org/wiki/xacro'>
     <xacro:arg name = 'robot_name' default = 'robot1'/>
-    <xacro:property name = 'robot_name' value = '${arg robot_name}'/>
+    <xacro:property name = 'prefix' value = '${arg robot_name}_'/>
     <!-- include files -->
     <xacro:include filename = 'robot_body.xacro'/>
-    <xacro:include filename = 'robot_peripherals.xacro'/>
-    <xacro:include filename = 'robot_gazebo_properties.xacro'/>
+    <!-- <xacro:include filename = 'robot_peripherals.xacro'/>
+    <xacro:include filename = 'robot_gazebo_properties.xacro'/> -->
 </robot>

Commit message: fixed the problem with inheritance. wrong quote type, and used '{}' instead of '()' for the property

File: mrs_robot_launcher/urdf/X3/robot.urdf.xacro (robot description, xacro)
@@ -1,9 +1,10 @@
 <?xml version='1.0'?>
 <robot name = 'robot' xmlns:xacro = 'http://www.ros.org/wiki/xacro'>
-    <xacro:arg name = 'robot_name' default = 'robot1'/>
-    <xacro:property name = 'prefix' value = '${arg robot_name}_'/>
+    <xacro:arg name = "robot_name" default = "robot1"/>
+    <xacro:property name = "prefix" value = "$(arg robot_name)_"/>
+    <DEBUG_MSG value = "Loading prefix value: ${prefix}"/>
     <!-- include files -->
     <xacro:include filename = 'robot_body.xacro'/>
-    <!-- <xacro:include filename = 'robot_peripherals.xacro'/>
-    <xacro:include filename = 'robot_gazebo_properties.xacro'/> -->
+    <xacro:include filename = 'robot_peripherals.xacro'/>
+    <!-- <xacro:include filename = 'robot_gazebo_properties.xacro'/> -->
 </robot>

Commit message: removed '_' from property 'prefix', this allows the property to be used in more than one way

File: mrs_robot_launcher/urdf/X3/robot.urdf.xacro (robot description, xacro)
@@ -2,5 +2,5 @@
 <robot name = 'robot' xmlns:xacro = 'http://www.ros.org/wiki/xacro'>
     <xacro:arg name = "robot_name" default = "robot1"/>
-    <xacro:property name = "prefix" value = "$(arg robot_name)_"/>
+    <xacro:property name = "prefix" value = "$(arg robot_name)"/>
     <DEBUG_MSG value = "Loading prefix value: ${prefix}"/>
     <!-- include files -->

Commit message: added argument and property for robot capability

File: mrs_robot_launcher/urdf/X3/robot.urdf.xacro (robot description, xacro)
@@ -1,6 +1,9 @@
 <?xml version='1.0'?>
 <robot name = 'robot' xmlns:xacro = 'http://www.ros.org/wiki/xacro'>
+    <!-- arguments and parameters -->
     <xacro:arg name = "robot_name" default = "robot1"/>
     <xacro:property name = "prefix" value = "$(arg robot_name)"/>
+    <xacro:arg name = "robot_capability" default = "depth"/>
+    <xacro:property name = "capability" value = "$(arg robot_capability)"/>
     <DEBUG_MSG value = "Loading prefix value: ${prefix}"/>
     <!-- include files -->
