Commit message: added ability to change colour of robot based on their capability

File: mrs_robot_launcher/urdf/X3/robot_gazebo_properties.xacro (robot description, xacro)
@@ -8,7 +8,14 @@
     <xacro:property name = 'kd' value = '7500'/>
     <!--            LINKS          -->
-    <gazebo reference = '${prefix}_chassis_link'>
-        <material>Gazebo/Green</material>
-    </gazebo>
+    <xacro:if value = "${capability == 'depth'}">
+        <gazebo reference = '${prefix}_chassis_link'>
+            <material>Gazebo/Blue</material>
+        </gazebo>
+    </xacro:if>
+    <xacro:if value = "${capability == 'thermal'}">
+        <gazebo reference = '${prefix}_chassis_link'>
+            <material>Gazebo/Red</material>
+        </gazebo>
+    </xacro:if>
     <gazebo reference = '${prefix}_front_right_wheel_link'>
         <material>Gazebo/Black</material>

Commit message: added support for different robot types based on the capabilities. 'depth' robots have the depth camera, need to figure out a way to add a different type -> should look into available sensors

File: mrs_robot_launcher/urdf/X3/robot_gazebo_properties.xacro (robot description, xacro)
@@ -88,31 +88,34 @@
         </sensor>
     </gazebo>
-    <gazebo reference = '${prefix}_camera_link'>
-        <material>Gazebo/Black</material>
-        <sensor name = 'camera' type = 'depth'>
-            <pose> 0 0 0 0 0 0 </pose>
-            <visualize>true</visualize>
-            <update_rate>10</update_rate>
-            <camera>
-                <horizontal_fov>1.019272283</horizontal_fov>
-                <vertical_fov>0.7941248097</vertical_fov>
-                <image>
-                    <format>R8G8B8</format>
-                    <width>640</width>
-                    <height>480</height>
-                </image>
-                <clip>
-                    <near>0.1</near>
-                    <far>8.0</far>
-                </clip>
-            </camera>
-            <plugin name = 'camera_controller' filename = 'libgazebo_ros_camera.so'>
-                <frame_name>${prefix}_camera_link_optical</frame_name>
-                <ros>
-                    <namespace>${prefix}</namespace>
-                </ros>
-            </plugin>
-        </sensor>
-    </gazebo>
+    <!-- for depth camera: -->
+    <xacro:if value = "${capability == 'depth'}">
+        <gazebo reference = '${prefix}_camera_link'>
+            <material>Gazebo/Black</material>
+            <sensor name = 'camera' type = 'depth'>
+                <pose> 0 0 0 0 0 0 </pose>
+                <visualize>true</visualize>
+                <update_rate>10</update_rate>
+                <camera>
+                    <horizontal_fov>1.019272283</horizontal_fov>
+                    <vertical_fov>0.7941248097</vertical_fov>
+                    <image>
+                        <format>R8G8B8</format>
+                        <width>640</width>
+                        <height>480</height>
+                    </image>
+                    <clip>
+                        <near>0.1</near>
+                        <far>8.0</far>
+                    </clip>
+                </camera>
+                <plugin name = 'camera_controller' filename = 'libgazebo_ros_camera.so'>
+                    <frame_name>${prefix}_camera_link_optical</frame_name>
+                    <ros>
+                        <namespace>${prefix}</namespace>
+                    </ros>
+                </plugin>
+            </sensor>
+        </gazebo>
+    </xacro:if>
     <!--            GAZEBO CONTROL           -->
     <gazebo>

File: mrs_robot_launcher/urdf/X3/robot_peripherals.xacro (robot description, xacro)
@@ -33,36 +33,38 @@
     </joint>
     <!-- camera link -->
-    <link name = '${prefix}_camera_link'>
-        <visual>
-            <origin xyz = '0 0 0' rpy = '0 0 0'/>
-            <geometry>
-                <mesh filename = 'file://$(find mrs_robot_launcher)/meshes/camera.STL'/>
-            </geometry>
-            <material name = 'black'/>
-        </visual>
-        <inertial>
-            <mass value = '0.30393'/>
-            <xacro:box_inertia
-                mass = '0.30393'
-                w = '0.06'
-                h = '0.05'
-                d = '0.165'
-            />
-        </inertial>
-    </link>
-    <!-- camera to chassis joint -->
-    <joint name = '${prefix}_camera_joint' type = 'fixed'>
-        <origin xyz = '0.057105 1.7948E-05 0.03755' rpy = '0 0 0'/>
-        <parent link = '${prefix}_chassis_link'/>
-        <child link = '${prefix}_camera_link'/>
-    </joint>
-    <!-- optical link for camera coordinate frame -->
-    <link name = '${prefix}_camera_link_optical'>
-    </link>
-    <!-- optical camera link to actual camera link joint: -->
-    <joint name = '${prefix}_camera_optical_joint' type = 'fixed'>
-        <origin xyz = '0 0 0' rpy = '-1.570796 0 -1.570796'/>
-        <parent link = '${prefix}_camera_link'/>
-        <child link = '${prefix}_camera_link_optical'/>
-    </joint>
+    <xacro:if value = "${capability == 'depth'}">
+        <link name = '${prefix}_camera_link'>
+            <visual>
+                <origin xyz = '0 0 0' rpy = '0 0 0'/>
+                <geometry>
+                    <mesh filename = 'file://$(find mrs_robot_launcher)/meshes/camera.STL'/>
+                </geometry>
+                <material name = 'black'/>
+            </visual>
+            <inertial>
+                <mass value = '0.30393'/>
+                <xacro:box_inertia
+                    mass = '0.30393'
+                    w = '0.06'
+                    h = '0.05'
+                    d = '0.165'
+                />
+            </inertial>
+        </link>
+        <!-- camera to chassis joint -->
+        <joint name = '${prefix}_camera_joint' type = 'fixed'>
+            <origin xyz = '0.057105 1.7948E-05 0.03755' rpy = '0 0 0'/>
+            <parent link = '${prefix}_chassis_link'/>
+            <child link = '${prefix}_camera_link'/>
+        </joint>
+        <!-- optical link for camera coordinate frame -->
+        <link name = '${prefix}_camera_link_optical'>
+        </link>
+        <!-- optical camera link to actual camera link joint: -->
+        <joint name = '${prefix}_camera_optical_joint' type = 'fixed'>
+            <origin xyz = '0 0 0' rpy = '-1.570796 0 -1.570796'/>
+            <parent link = '${prefix}_camera_link'/>
+            <child link = '${prefix}_camera_link_optical'/>
+        </joint>
+    </xacro:if>
 </robot>

Commit message: added ability to process thermal robots separately. added a thermal camera, realized it was just the lid and switched back to the depth. need to add thermal mesh and orient it correctly

File: mrs_robot_launcher/urdf/X3/robot_gazebo_properties.xacro (robot description, xacro)
@@ -90,5 +90,5 @@
     <!-- for depth camera: -->
     <xacro:if value = "${capability == 'depth'}">
-        <gazebo reference = '${prefix}_camera_link'>
+        <gazebo reference = '${prefix}_depth_camera_link'>
             <material>Gazebo/Black</material>
             <sensor name = 'camera' type = 'depth'>

File: mrs_robot_launcher/urdf/X3/robot_peripherals.xacro (robot description, xacro)
@@ -32,7 +32,7 @@
         <child link = '${prefix}_lidar_link'/>
     </joint>
-    <!-- camera link -->
+    <!-- depth camera link -->
     <xacro:if value = "${capability == 'depth'}">
-        <link name = '${prefix}_camera_link'>
+        <link name = '${prefix}_depth_camera_link'>
             <visual>
                 <origin xyz = '0 0 0' rpy = '0 0 0'/>
@@ -52,18 +52,45 @@
             </inertial>
         </link>
-        <!-- camera to chassis joint -->
+        <!-- depth camera to chassis joint -->
         <joint name = '${prefix}_camera_joint' type = 'fixed'>
             <origin xyz = '0.057105 1.7948E-05 0.03755' rpy = '0 0 0'/>
             <parent link = '${prefix}_chassis_link'/>
-            <child link = '${prefix}_camera_link'/>
+            <child link = '${prefix}_depth_camera_link'/>
         </joint>
-        <!-- optical link for camera coordinate frame -->
-        <link name = '${prefix}_camera_link_optical'>
+        <!-- optical link for depth camera coordinate frame -->
+        <link name = '${prefix}_depth_camera_link_optical'>
         </link>
-        <!-- optical camera link to actual camera link joint: -->
+        <!-- optical depth camera link to actual depth camera link joint: -->
         <joint name = '${prefix}_camera_optical_joint' type = 'fixed'>
             <origin xyz = '0 0 0' rpy = '-1.570796 0 -1.570796'/>
-            <parent link = '${prefix}_camera_link'/>
-            <child link = '${prefix}_camera_link_optical'/>
+            <parent link = '${prefix}_depth_camera_link'/>
+            <child link = '${prefix}_depth_camera_link_optical'/>
+        </joint>
+    </xacro:if>
+    <!-- thermal camera link -->
+    <xacro:if value = "${capability == 'thermal'}">
+        <link name = "${prefix}_thermal_camera_link">
+            <visual>
+                <origin xyz = '0 0 0' rpy = '0 0 0'/>
+                <geometry>
+                    <mesh filename = 'file://$(find mrs_robot_launcher)/meshes/camera.STL'/>
+                </geometry>
+                <material name = 'black'/>
+            </visual>
+        </link>
+        <!-- thermal camera to chassis joint -->
+        <joint name = '${prefix}_thermal_camera_joint' type = 'fixed'>
+            <origin xyz = '0.057105 1.7948E-05 0.03755' rpy = '0 0 0'/>
+            <parent link = '${prefix}_chassis_link'/>
+            <child link = '${prefix}_thermal_camera_link'/>
+        </joint>
+        <!-- optical link for depth camera coordinate frame -->
+        <link name = '${prefix}_thermal_camera_link_optical'>
+        </link>
+        <!-- optical thermal camera link to actual thermal camera link joint: -->
+        <joint name = '${prefix}_camera_optical_joint' type = 'fixed'>
+            <origin xyz = '0 0 0' rpy = '-1.570796 0 -1.570796'/>
+            <parent link = '${prefix}_thermal_camera_link'/>
+            <child link = '${prefix}_thermal_camera_link_optical'/>
         </joint>
     </xacro:if>

Commit message: added thermal camera section with base camera plugin. need to remount camera to actual optical frame and separate visual from optical frame further

File: mrs_robot_launcher/urdf/X3/robot_gazebo_properties.xacro (robot description, xacro)
@@ -88,9 +88,9 @@
         </sensor>
     </gazebo>
-    <!-- for depth camera: -->
+    <!-- for depth camera -->
     <xacro:if value = "${capability == 'depth'}">
         <gazebo reference = '${prefix}_depth_camera_link'>
             <material>Gazebo/Black</material>
-            <sensor name = 'camera' type = 'depth'>
+            <sensor name = 'depth_camera' type = 'depth'>
                 <pose> 0 0 0 0 0 0 </pose>
                 <visualize>true</visualize>
@@ -109,6 +109,36 @@
                     </clip>
                 </camera>
-                <plugin name = 'camera_controller' filename = 'libgazebo_ros_camera.so'>
-                    <frame_name>${prefix}_camera_link_optical</frame_name>
+                <plugin name = 'depth_camera_controller' filename = 'libgazebo_ros_camera.so'>
+                    <frame_name>${prefix}_depth_camera_link_optical</frame_name>
+                    <ros>
+                        <namespace>${prefix}</namespace>
+                    </ros>
+                </plugin>
+            </sensor>
+        </gazebo>
+    </xacro:if>
+    <!-- for thermal camera -->
+    <xacro:if value = "${capability == 'thermal'}">
+        <gazebo reference = '${prefix}_thermal_camera_link'>
+            <material>Gazebo/Black</material>
+            <sensor name = "thermal_cam" type = "camera">
+                <pose>0 0 0 0 0 0</pose>
+                <visualize>true</visualize>
+                <update_rate>10</update_rate>
+                <camera>
+                    <horizontal_fov>0.8499753</horizontal_fov>
+                    <vertical_fov>0.6736971</vertical_fov>
+                    <image>
+                        <format>R8G8B8</format>
+                        <width>640</width>
+                        <height>512</height>
+                    </image>
+                    <clip>
+                        <near>0.1</near>
+                        <far>8.0</far>
+                    </clip>
+                </camera>
+                <plugin name = 'thermal_camera_controller' filename = 'libgazebo_ros_camera.so'>
+                    <frame_name>${prefix}_thermal_camera_link_optical</frame_name>
                     <ros>
                         <namespace>${prefix}</namespace>
@@ -120,5 +150,5 @@
     <!--            GAZEBO CONTROL           -->
     <gazebo>
-        <plugin name = 'omni_robot' filename = 'libgazebo_ros_omni_drive.so'>
+        <plugin name = 'omni_robot_controller' filename = 'libgazebo_ros_omni_drive.so'>
             <!-- namespacing -->
             <ros>
