Commit message: prefixed links & joints

File: mrs_robot_launcher/urdf/X3/robot_peripherals.xacro (robot description, xacro)
@@ -3,5 +3,5 @@
     <!--            PERIPHERALS & JOINTS             -->
     <!-- lidar link -->
-    <link name = 'lidar_link'>
+    <link name = '${robot_name}_lidar_link'>
         <visual>
             <origin xyz = '0 0 0' rpy = '1.570796 0 1.570796'/>
@@ -27,11 +27,11 @@
     </link>
     <!-- lidar to chassis joint -->
-    <joint name = 'lidar_joint' type = 'fixed'>
+    <joint name = '${robot_name}_lidar_joint' type = 'fixed'>
         <origin xyz = '0.0405 5.25826986680105E-05 0.08285' rpy = '0 0 0'/>
-        <parent link = 'chassis_link'/>
-        <child link = 'lidar_link'/>
+        <parent link = '${robot_name}_chassis_link'/>
+        <child link = '${robot_name}_lidar_link'/>
     </joint>
     <!-- camera link -->
-    <link name = 'camera_link'>
+    <link name = '${robot_name}_camera_link'>
         <visual>
             <origin xyz = '0 0 0' rpy = '0 0 0'/>
@@ -52,17 +52,17 @@
     </link>
     <!-- camera to chassis joint -->
-    <joint name = 'camera_joint' type = 'fixed'>
+    <joint name = '${robot_name}_camera_joint' type = 'fixed'>
         <origin xyz = '0.057105 1.7948E-05 0.03755' rpy = '0 0 0'/>
-        <parent link = 'chassis_link'/>
-        <child link = 'camera_link'/>
+        <parent link = '${robot_name}_chassis_link'/>
+        <child link = '${robot_name}_camera_link'/>
     </joint>
     <!-- optical link for camera coordinate frame -->
-    <link name = 'camera_link_optical'>
+    <link name = '${robot_name}_camera_link_optical'>
     </link>
     <!-- optical camera link to actual camera link joint: -->
-    <joint name = 'camera_optical_joint' type = 'fixed'>
+    <joint name = '${robot_name}_camera_optical_joint' type = 'fixed'>
         <origin xyz = '0 0 0' rpy = '-1.570796 0 -1.570796'/>
-        <parent link = 'camera_link'/>
-        <child link = 'camera_link_optical'/>
+        <parent link = '${robot_name}_camera_link'/>
+        <child link = '${robot_name}_camera_link_optical'/>
     </joint>
 </robot>

Commit message: added the thermal camera assembly and correctly oriented both the camera and optical frame

File: mrs_robot_launcher/urdf/X3/robot_peripherals.xacro (robot description, xacro)
@@ -74,5 +74,5 @@
                 <origin xyz = '0 0 0' rpy = '0 0 0'/>
                 <geometry>
-                    <mesh filename = 'file://$(find mrs_robot_launcher)/meshes/camera.STL'/>
+                    <mesh filename = 'file://$(find mrs_robot_launcher)/meshes/thermal_cam_assembly.STL' scale = '0.001 0.001 0.001'/>
                 </geometry>
                 <material name = 'black'/>
@@ -81,5 +81,6 @@
         <!-- thermal camera to chassis joint -->
         <joint name = '${prefix}_thermal_camera_joint' type = 'fixed'>
-            <origin xyz = '0.057105 1.7948E-05 0.03755' rpy = '0 0 0'/>
+            <!-- <origin xyz = '0.057105 1.7948E-05 0.03755' rpy = '0 0 0'/> -->
+            <origin xyz = '0.08 0 0.010' rpy = '1.570796 0 1.570796'/>
             <parent link = '${prefix}_chassis_link'/>
             <child link = '${prefix}_thermal_camera_link'/>
@@ -90,5 +91,5 @@
         <!-- optical thermal camera link to actual thermal camera link joint: -->
         <joint name = '${prefix}_camera_optical_joint' type = 'fixed'>
-            <origin xyz = '0 0 0' rpy = '-1.570796 0 -1.570796'/>
+            <origin xyz = '0 0.0375 0.02' rpy = '0 0 -1.570796'/>
             <parent link = '${prefix}_thermal_camera_link'/>
             <child link = '${prefix}_thermal_camera_link_optical'/>

Commit message: moved optical frame OUTSIDE of visual camera, fixing occlusion

File: mrs_robot_launcher/urdf/X3/robot_peripherals.xacro (robot description, xacro)
@@ -63,5 +63,5 @@
         <!-- optical depth camera link to actual depth camera link joint: -->
         <joint name = '${prefix}_camera_optical_joint' type = 'fixed'>
-            <origin xyz = '0 0 0' rpy = '-1.570796 0 -1.570796'/>
+            <origin xyz = '0.019 0 0' rpy = '-1.570796 0 -1.570796'/>
             <parent link = '${prefix}_depth_camera_link'/>
             <child link = '${prefix}_depth_camera_link_optical'/>

Commit message: moved visual representation of cameras to where the optical link is. changed naming convention for optical link. changed optical link to have the correct frame: Z-axis forward, X-axis right, Y-axis down

File: mrs_robot_launcher/urdf/X3/robot_peripherals.xacro (robot description, xacro)
@@ -36,5 +36,5 @@
         <link name = '${prefix}_depth_camera_link'>
             <visual>
-                <origin xyz = '0 0 0' rpy = '0 0 0'/>
+                <origin xyz = '-0.018 0 0' rpy = '0 0 0'/>
                 <geometry>
                     <mesh filename = 'file://$(find mrs_robot_launcher)/meshes/camera.STL'/>
@@ -54,16 +54,16 @@
         <!-- depth camera to chassis joint -->
         <joint name = '${prefix}_camera_joint' type = 'fixed'>
-            <origin xyz = '0.057105 1.7948E-05 0.03755' rpy = '0 0 0'/>
+            <origin xyz = '0.075105 1.7948E-05 0.03755' rpy = '0 0 0'/>
             <parent link = '${prefix}_chassis_link'/>
             <child link = '${prefix}_depth_camera_link'/>
         </joint>
         <!-- optical link for depth camera coordinate frame -->
-        <link name = '${prefix}_depth_camera_link_optical'>
+        <link name = '${prefix}_depth_camera_optical_link'>
         </link>
         <!-- optical depth camera link to actual depth camera link joint: -->
         <joint name = '${prefix}_camera_optical_joint' type = 'fixed'>
-            <origin xyz = '0.019 0 0' rpy = '-1.570796 0 -1.570796'/>
+            <origin xyz = '0 0 0' rpy = '-1.570796 0 -1.570796'/>
             <parent link = '${prefix}_depth_camera_link'/>
-            <child link = '${prefix}_depth_camera_link_optical'/>
+            <child link = '${prefix}_depth_camera_optical_link'/>
         </joint>
     </xacro:if>
@@ -72,5 +72,5 @@
         <link name = "${prefix}_thermal_camera_link">
             <visual>
-                <origin xyz = '0 0 0' rpy = '0 0 0'/>
+                <origin xyz = '-0.02 0 -0.0375' rpy = '1.570796 0 1.570796'/>
                 <geometry>
                     <mesh filename = 'file://$(find mrs_robot_launcher)/meshes/thermal_cam_assembly.STL' scale = '0.001 0.001 0.001'/>
@@ -82,16 +82,16 @@
         <joint name = '${prefix}_thermal_camera_joint' type = 'fixed'>
             <!-- <origin xyz = '0.057105 1.7948E-05 0.03755' rpy = '0 0 0'/> -->
-            <origin xyz = '0.08 0 0.010' rpy = '1.570796 0 1.570796'/>
+            <origin xyz = '0.1 0 0.0475' rpy = '0 0 0'/>
             <parent link = '${prefix}_chassis_link'/>
             <child link = '${prefix}_thermal_camera_link'/>
         </joint>
         <!-- optical link for depth camera coordinate frame -->
-        <link name = '${prefix}_thermal_camera_link_optical'>
+        <link name = '${prefix}_thermal_camera_optical_link'>
         </link>
         <!-- optical thermal camera link to actual thermal camera link joint: -->
         <joint name = '${prefix}_camera_optical_joint' type = 'fixed'>
-            <origin xyz = '0 0.0375 0.02' rpy = '0 0 -1.570796'/>
+            <origin xyz = '0 0 0' rpy = '-1.570796 0 -1.570796'/>
             <parent link = '${prefix}_thermal_camera_link'/>
-            <child link = '${prefix}_thermal_camera_link_optical'/>
+            <child link = '${prefix}_thermal_camera_optical_link'/>
         </joint>
     </xacro:if>
