Commit message: changed package name

File: mrs_robot_launcher/urdf/X3/robot_body.xacro (robot description, xacro)
@@ -46,5 +46,5 @@
             <origin xyz = '0 0 0' rpy = '0 0 0'/>
             <geometry>
-                <mesh filename = 'file://$(find sim_robot_description)/meshes/chassis.STL'/>
+                <mesh filename = 'file://$(find mrs_robot_launcher)/meshes/chassis.STL'/>
             </geometry>
             <material name = 'green'/>
@@ -78,5 +78,5 @@
             <origin xyz = '0 0 0' rpy = '1.570796 0 0'/>
             <geometry>
-                <mesh filename = 'file://$(find sim_robot_description)/meshes/front_right_wheel.STL'/>
+                <mesh filename = 'file://$(find mrs_robot_launcher)/meshes/front_right_wheel.STL'/>
             </geometry>
             <material name = 'black'/>
@@ -110,5 +110,5 @@
             <origin xyz = '0 0 0' rpy = '1.570796 0 0'/>
             <geometry>
-                <mesh filename = 'file://$(find sim_robot_description)/meshes/front_left_wheel.STL'/>
+                <mesh filename = 'file://$(find mrs_robot_launcher)/meshes/front_left_wheel.STL'/>
             </geometry>
             <material name = 'black'/>
@@ -142,5 +142,5 @@
             <origin xyz = '0 0 0' rpy = '1.570796 0 0'/>
             <geometry>
-                <mesh filename = 'file://$(find sim_robot_description)/meshes/back_right_wheel.STL'/>
+                <mesh filename = 'file://$(find mrs_robot_launcher)/meshes/back_right_wheel.STL'/>
             </geometry>
             <material name = 'black'/>
@@ -174,5 +174,5 @@
             <origin xyz = '0 0 0' rpy = '1.570796 0 0'/>
             <geometry>
-                <mesh filename = 'file://$(find sim_robot_description)/meshes/back_left_wheel.STL'/>
+                <mesh filename = 'file://$(find mrs_robot_launcher)/meshes/back_left_wheel.STL'/>
             </geometry>
             <material name = 'black'/>

File: mrs_robot_launcher/urdf/X3/robot_peripherals.xacro (robot description, xacro)
@@ -7,5 +7,5 @@
             <origin xyz = '0 0 0' rpy = '1.570796 0 1.570796'/>
             <geometry>
-                <mesh filename = 'file://$(find sim_robot_description)/meshes/lidar.STL' scale = '0.001 0.001 0.001'/>
+                <mesh filename = 'file://$(find mrs_robot_launcher)/meshes/lidar.STL' scale = '0.001 0.001 0.001'/>
             </geometry>
             <material name = 'black'/>
@@ -37,5 +37,5 @@
             <origin xyz = '0 0 0' rpy = '0 0 0'/>
             <geometry>
-                <mesh filename = 'file://$(find sim_robot_description)/meshes/camera.STL'/>
+                <mesh filename = 'file://$(find mrs_robot_launcher)/meshes/camera.STL'/>
             </geometry>
             <material name = 'black'/>

Commit message: prefixed links & joints

File: mrs_robot_launcher/urdf/X3/robot_body.xacro (robot description, xacro)
@@ -39,8 +39,8 @@
     <!-- BASE LINK & CHASSIS LINK -->
     <!-- base link -->
-    <link name = 'base_link'>
+    <link name = '${robot_name}_base_link'>
     </link>
     <!-- chassis link -->
-    <link name = 'chassis_link'>
+    <link name = '${robot_name}_chassis_link'>
         <visual>
             <origin xyz = '0 0 0' rpy = '0 0 0'/>
@@ -67,12 +67,12 @@
     </link>
     <!-- chassis to base joint -->
-    <joint name = 'base_joint' type = 'fixed'>
-        <parent link = 'base_link'/>
-        <child link = 'chassis_link'/>
+    <joint name = '${robot_name}_base_joint' type = 'fixed'>
+        <parent link = '${robot_name}_base_link'/>
+        <child link = '${robot_name}_chassis_link'/>
         <origin xyz = '0 0 0.07115' rpy = '0 0 0'/> <!-- origin offset of 0.07115 -->
     </joint>
     <!-- WHEEL LINKS & JOINTS -->
     <!-- front right wheel link -->
-    <link name = 'front_right_wheel_link'>
+    <link name = '${robot_name}_front_right_wheel_link'>
         <visual>
             <origin xyz = '0 0 0' rpy = '1.570796 0 0'/>
@@ -98,13 +98,13 @@
     </link>
     <!-- front right wheel to chassis joint -->
-    <joint name = 'front_right_joint' type = 'continuous'>
+    <joint name = '${robot_name}_front_right_joint' type = 'continuous'>
         <origin xyz = '0.08 -0.08475 -0.0389' rpy = '0 0 0'/>
-        <parent link = 'chassis_link'/>
-        <child link = 'front_right_wheel_link'/>
+        <parent link = '${robot_name}_chassis_link'/>
+        <child link = '${robot_name}_front_right_wheel_link'/>
         <axis xyz = '0 1 0' rpy = '0 0 0'/>
         <dynamics damping = '${d}'/>
     </joint>
     <!-- front left wheel link -->
-    <link name = 'front_left_wheel_link'>
+    <link name = '${robot_name}_front_left_wheel_link'>
         <visual>
             <origin xyz = '0 0 0' rpy = '1.570796 0 0'/>
@@ -130,13 +130,13 @@
     </link>
     <!-- front left wheel to chassis joint -->
-    <joint name = 'front_left_joint' type = 'continuous'>
+    <joint name = '${robot_name}_front_left_joint' type = 'continuous'>
         <origin xyz = '0.08 0.08475 -0.0389' rpy = '0 0 0'/>
-        <parent link = 'chassis_link'/>
-        <child link = 'front_left_wheel_link'/>
+        <parent link = '${robot_name}_chassis_link'/>
+        <child link = '${robot_name}_front_left_wheel_link'/>
         <axis xyz = '0 1 0' rpy = '0 0 0'/>
         <dynamics damping = '${d}'/>
     </joint>
     <!-- back right wheel link -->
-    <link name = 'back_right_wheel_link'>
+    <link name = '${robot_name}_back_right_wheel_link'>
         <visual>
             <origin xyz = '0 0 0' rpy = '1.570796 0 0'/>
@@ -162,13 +162,13 @@
     </link>
     <!-- back right wheel to chassis joint -->
-    <joint name = 'back_right_joint' type = 'continuous'>
+    <joint name = '${robot_name}_back_right_joint' type = 'continuous'>
         <origin xyz = '-0.08 -0.08475 -0.0389' rpy = '0 0 0'/>   <!-- z was -0.03946 -->
-        <parent link = 'chassis_link'/>
-        <child link = 'back_right_wheel_link'/>
+        <parent link = '${robot_name}_chassis_link'/>
+        <child link = '${robot_name}_back_right_wheel_link'/>
         <axis xyz = '0 1 0' rpy = '0 0 0'/>
         <dynamics damping = '${d}'/>
     </joint>
     <!-- back left wheel link -->
-    <link name = 'back_left_wheel_link'>
+    <link name = '${robot_name}_back_left_wheel_link'>
         <visual>
             <origin xyz = '0 0 0' rpy = '1.570796 0 0'/>
@@ -194,8 +194,8 @@
     </link>
     <!-- back left wheel to chassis joint -->
-    <joint name = 'back_left_joint' type = 'continuous'>
+    <joint name = '${robot_name}_back_left_joint' type = 'continuous'>
         <origin xyz = '-0.08 0.08475 -0.0389' rpy = '0 0 0'/> <!-- z was -0.03954 -->
-        <parent link = 'chassis_link'/>
-        <child link = 'back_left_wheel_link'/>
+        <parent link = '${robot_name}_chassis_link'/>
+        <child link = '${robot_name}_back_left_wheel_link'/>
         <axis xyz = '0 1 0' rpy = '0 0 0'/>
         <dynamics damping = '${d}'/>

Commit message: added prefixing

File: mrs_robot_launcher/urdf/X3/robot_body.xacro (robot description, xacro)
@@ -39,8 +39,8 @@
     <!-- BASE LINK & CHASSIS LINK -->
     <!-- base link -->
-    <link name = '${robot_name}_base_link'>
+    <link name = '${prefix}base_link'>
     </link>
     <!-- chassis link -->
-    <link name = '${robot_name}_chassis_link'>
+    <link name = '${prefix}chassis_link'>
         <visual>
             <origin xyz = '0 0 0' rpy = '0 0 0'/>
@@ -67,12 +67,12 @@
     </link>
     <!-- chassis to base joint -->
-    <joint name = '${robot_name}_base_joint' type = 'fixed'>
-        <parent link = '${robot_name}_base_link'/>
-        <child link = '${robot_name}_chassis_link'/>
+    <joint name = '${prefix}base_joint' type = 'fixed'>
+        <parent link = '${prefix}base_link'/>
+        <child link = '${prefix}chassis_link'/>
         <origin xyz = '0 0 0.07115' rpy = '0 0 0'/> <!-- origin offset of 0.07115 -->
     </joint>
     <!-- WHEEL LINKS & JOINTS -->
     <!-- front right wheel link -->
-    <link name = '${robot_name}_front_right_wheel_link'>
+    <link name = '${prefix}front_right_wheel_link'>
         <visual>
             <origin xyz = '0 0 0' rpy = '1.570796 0 0'/>
@@ -98,13 +98,13 @@
     </link>
     <!-- front right wheel to chassis joint -->
-    <joint name = '${robot_name}_front_right_joint' type = 'continuous'>
+    <joint name = '${prefix}front_right_joint' type = 'continuous'>
         <origin xyz = '0.08 -0.08475 -0.0389' rpy = '0 0 0'/>
-        <parent link = '${robot_name}_chassis_link'/>
-        <child link = '${robot_name}_front_right_wheel_link'/>
+        <parent link = '${prefix}chassis_link'/>
+        <child link = '${prefix}front_right_wheel_link'/>
         <axis xyz = '0 1 0' rpy = '0 0 0'/>
         <dynamics damping = '${d}'/>
     </joint>
     <!-- front left wheel link -->
-    <link name = '${robot_name}_front_left_wheel_link'>
+    <link name = '${prefix}front_left_wheel_link'>
         <visual>
             <origin xyz = '0 0 0' rpy = '1.570796 0 0'/>
@@ -130,13 +130,13 @@
     </link>
     <!-- front left wheel to chassis joint -->
-    <joint name = '${robot_name}_front_left_joint' type = 'continuous'>
+    <joint name = '${prefix}front_left_joint' type = 'continuous'>
         <origin xyz = '0.08 0.08475 -0.0389' rpy = '0 0 0'/>
-        <parent link = '${robot_name}_chassis_link'/>
-        <child link = '${robot_name}_front_left_wheel_link'/>
+        <parent link = '${prefix}chassis_link'/>
+        <child link = '${prefix}front_left_wheel_link'/>
         <axis xyz = '0 1 0' rpy = '0 0 0'/>
         <dynamics damping = '${d}'/>
     </joint>
     <!-- back right wheel link -->
-    <link name = '${robot_name}_back_right_wheel_link'>
+    <link name = '${prefix}back_right_wheel_link'>
         <visual>
             <origin xyz = '0 0 0' rpy = '1.570796 0 0'/>
@@ -162,13 +162,13 @@
     </link>
     <!-- back right wheel to chassis joint -->
-    <joint name = '${robot_name}_back_right_joint' type = 'continuous'>
+    <joint name = '${prefix}back_right_joint' type = 'continuous'>
         <origin xyz = '-0.08 -0.08475 -0.0389' rpy = '0 0 0'/>   <!-- z was -0.03946 -->
-        <parent link = '${robot_name}_chassis_link'/>
-        <child link = '${robot_name}_back_right_wheel_link'/>
+        <parent link = '${prefix}chassis_link'/>
+        <child link = '${prefix}back_right_wheel_link'/>
         <axis xyz = '0 1 0' rpy = '0 0 0'/>
         <dynamics damping = '${d}'/>
     </joint>
     <!-- back left wheel link -->
-    <link name = '${robot_name}_back_left_wheel_link'>
+    <link name = '${prefix}back_left_wheel_link'>
         <visual>
             <origin xyz = '0 0 0' rpy = '1.570796 0 0'/>
@@ -194,8 +194,8 @@
     </link>
     <!-- back left wheel to chassis joint -->
-    <joint name = '${robot_name}_back_left_joint' type = 'continuous'>
+    <joint name = '${prefix}back_left_joint' type = 'continuous'>
         <origin xyz = '-0.08 0.08475 -0.0389' rpy = '0 0 0'/> <!-- z was -0.03954 -->
-        <parent link = '${robot_name}_chassis_link'/>
-        <child link = '${robot_name}_back_left_wheel_link'/>
+        <parent link = '${prefix}chassis_link'/>
+        <child link = '${prefix}back_left_wheel_link'/>
         <axis xyz = '0 1 0' rpy = '0 0 0'/>
         <dynamics damping = '${d}'/>

File: mrs_robot_launcher/urdf/X3/robot_gazebo_properties.xacro (robot description, xacro)
@@ -8,48 +8,48 @@
     <xacro:property name = 'kd' value = '7500'/>
     <!--            LINKS          -->
-    <gazebo reference = '${robot_name}_base_link'>
+    <gazebo reference = '${prefix}base_link'>
         <material>Gazebo/Green</material>
     </gazebo>
-    <gazebo reference = '${robot_name}_front_right_wheel_link'>
+    <gazebo reference = '${prefix}front_right_wheel_link'>
         <material>Gazebo/Black</material>
         <pose>0 0 0 0 0 0</pose>
         <mu1 value = '${mu1}' />
         <mu2 value = '${mu2}' />
-        <fdir1 gz:expressed_in='${robot_name}_base_link'>1 1 0</fdir1>
+        <fdir1 gz:expressed_in='${prefix}base_link'>1 1 0</fdir1>
         <minDepth>${minDepth}</minDepth>
         <kp>${kp}</kp>
         <kd>${kd}</kd>
     </gazebo>
-    <gazebo reference = '${robot_name}_front_left_wheel_link'>
+    <gazebo reference = '${prefix}front_left_wheel_link'>
         <material>Gazebo/Black</material>
         <pose>0 0 0 0 0 0</pose>
         <mu1 value = '${mu1}' />
         <mu2 value = '${mu2}' />
-        <fdir1 gz:expressed_in='${robot_name}_base_link'>-1 1 0</fdir1>
+        <fdir1 gz:expressed_in='${prefix}base_link'>-1 1 0</fdir1>
         <minDepth>${minDepth}</minDepth>
         <kp>${kp}</kp>
         <kd>${kd}</kd>
     </gazebo>
-    <gazebo reference = '${robot_name}_back_right_wheel_link'>
+    <gazebo reference = '${prefix}back_right_wheel_link'>
         <material>Gazebo/Black</material>
         <pose>0 0 0 0 0 0</pose>
         <mu1 value = '${mu1}' />
         <mu2 value = '${mu2}' />
-        <fdir1 gz:expressed_in='${robot_name}_base_link'>1 -1 0</fdir1>
+        <fdir1 gz:expressed_in='${prefix}base_link'>1 -1 0</fdir1>
         <minDepth>${minDepth}</minDepth>
         <kp>${kp}</kp>
         <kd>${kd}</kd>
     </gazebo>
-    <gazebo reference = '${robot_name}_back_left_wheel_link'>
+    <gazebo reference = '${prefix}back_left_wheel_link'>
         <material>Gazebo/Black</material>
         <pose>0 0 0 0 0 0</pose>
         <mu1 value = '${mu1}' />
         <mu2 value = '${mu2}' />
-        <fdir1 gz:expressed_in='${robot_name}_base_link'>-1 -1 0</fdir1>
+        <fdir1 gz:expressed_in='${prefix}base_link'>-1 -1 0</fdir1>
         <minDepth>${minDepth}</minDepth>
         <kp>${kp}</kp>
         <kd>${kd}</kd>
     </gazebo>
-    <gazebo reference = '${robot_name}_lidar_link'>
+    <gazebo reference = '${prefix}lidar_link'>
         <material>Gazebo/Black</material>
         <sensor name = 'lidar' type = 'ray'>
@@ -76,9 +76,9 @@
                 </ros>
                 <output_type>sensor_msgs/LaserScan</output_type>
-                <frame_name>${robot_name}_lidar_link</frame_name>
+                <frame_name>${prefix}lidar_link</frame_name>
             </plugin>
         </sensor>
     </gazebo>
-    <gazebo reference = '${robot_name}_camera_link'>
+    <gazebo reference = '${prefix}camera_link'>
         <material>Gazebo/Black</material>
         <sensor name = 'camera' type = 'depth'>
@@ -100,5 +100,5 @@
             </camera>
             <plugin name = 'camera_controller' filename = 'libgazebo_ros_camera.so'>
-                <frame_name>${robot_name}_camera_link_optical</frame_name>
+                <frame_name>${prefix}camera_link_optical</frame_name>
             </plugin>
         </sensor>
@@ -111,13 +111,13 @@
             <odometryFrame>odom</odometryFrame>
             <odometryRate>250.0</odometryRate>
-            <robotBaseFrame>${robot_name}_base_link</robotBaseFrame>
+            <robotBaseFrame>${prefix}base_link</robotBaseFrame>
             <publish_wheel_tf>true</publish_wheel_tf>
             <wheel_radius>0.0325</wheel_radius>
             <base_length>0.16</base_length>
             <base_width>0.1695</base_width>
-            <front_right_joint>${robot_name}_front_right_joint</front_right_joint>
-            <front_left_joint>${robot_name}_front_left_joint</front_left_joint>
-            <rear_right_joint>${robot_name}_back_right_joint</rear_right_joint>
-            <rear_left_joint>${robot_name}_back_left_joint</rear_left_joint>
+            <front_right_joint>${prefix}front_right_joint</front_right_joint>
+            <front_left_joint>${prefix}front_left_joint</front_left_joint>
+            <rear_right_joint>${prefix}back_right_joint</rear_right_joint>
+            <rear_left_joint>${prefix}back_left_joint</rear_left_joint>
             <wheel_max_speed>7.50</wheel_max_speed>
             <wheel_acceleration>7.50</wheel_acceleration>

File: mrs_robot_launcher/urdf/X3/robot_peripherals.xacro (robot description, xacro)
@@ -3,5 +3,5 @@
     <!--            PERIPHERALS & JOINTS             -->
     <!-- lidar link -->
-    <link name = '${robot_name}_lidar_link'>
+    <link name = '${prefix}lidar_link'>
         <visual>
             <origin xyz = '0 0 0' rpy = '1.570796 0 1.570796'/>
@@ -27,11 +27,11 @@
     </link>
     <!-- lidar to chassis joint -->
-    <joint name = '${robot_name}_lidar_joint' type = 'fixed'>
+    <joint name = '${prefix}lidar_joint' type = 'fixed'>
         <origin xyz = '0.0405 5.25826986680105E-05 0.08285' rpy = '0 0 0'/>
-        <parent link = '${robot_name}_chassis_link'/>
-        <child link = '${robot_name}_lidar_link'/>
+        <parent link = '${prefix}chassis_link'/>
+        <child link = '${prefix}lidar_link'/>
     </joint>
     <!-- camera link -->
-    <link name = '${robot_name}_camera_link'>
+    <link name = '${prefix}camera_link'>
         <visual>
             <origin xyz = '0 0 0' rpy = '0 0 0'/>
@@ -52,17 +52,17 @@
     </link>
     <!-- camera to chassis joint -->
-    <joint name = '${robot_name}_camera_joint' type = 'fixed'>
+    <joint name = '${prefix}camera_joint' type = 'fixed'>
         <origin xyz = '0.057105 1.7948E-05 0.03755' rpy = '0 0 0'/>
-        <parent link = '${robot_name}_chassis_link'/>
-        <child link = '${robot_name}_camera_link'/>
+        <parent link = '${prefix}chassis_link'/>
+        <child link = '${prefix}camera_link'/>
     </joint>
     <!-- optical link for camera coordinate frame -->
-    <link name = '${robot_name}_camera_link_optical'>
+    <link name = '${prefix}camera_link_optical'>
     </link>
     <!-- optical camera link to actual camera link joint: -->
-    <joint name = '${robot_name}_camera_optical_joint' type = 'fixed'>
+    <joint name = '${prefix}camera_optical_joint' type = 'fixed'>
         <origin xyz = '0 0 0' rpy = '-1.570796 0 -1.570796'/>
-        <parent link = '${robot_name}_camera_link'/>
-        <child link = '${robot_name}_camera_link_optical'/>
+        <parent link = '${prefix}camera_link'/>
+        <child link = '${prefix}camera_link_optical'/>
     </joint>
 </robot>
