Commit message: added '_' to reflect changes in property 'prefix'

File: mrs_robot_launcher/urdf/X3/robot_body.xacro (robot description, xacro)
@@ -39,8 +39,8 @@
     <!-- BASE LINK & CHASSIS LINK -->
     <!-- base link -->
-    <link name = '${prefix}base_link'>
+    <link name = '${prefix}_base_link'>
     </link>
     <!-- chassis link -->
-    <link name = '${prefix}chassis_link'>
+    <link name = '${prefix}_chassis_link'>
         <visual>
             <origin xyz = '0 0 0' rpy = '0 0 0'/>
@@ -67,12 +67,12 @@
     </link>
     <!-- chassis to base joint -->
-    <joint name = '${prefix}base_joint' type = 'fixed'>
-        <parent link = '${prefix}base_link'/>
-        <child link = '${prefix}chassis_link'/>
+    <joint name = '${prefix}_base_joint' type = 'fixed'>
+        <parent link = '${prefix}_base_link'/>
+        <child link = '${prefix}_chassis_link'/>
         <origin xyz = '0 0 0.07115' rpy = '0 0 0'/> <!-- origin offset of 0.07115 -->
     </joint>
     <!-- WHEEL LINKS & JOINTS -->
     <!-- front right wheel link -->
-    <link name = '${prefix}front_right_wheel_link'>
+    <link name = '${prefix}_front_right_wheel_link'>
         <visual>
             <origin xyz = '0 0 0' rpy = '1.570796 0 0'/>
@@ -98,13 +98,13 @@
     </link>
     <!-- front right wheel to chassis joint -->
-    <joint name = '${prefix}front_right_joint' type = 'continuous'>
+    <joint name = '${prefix}_front_right_joint' type = 'continuous'>
         <origin xyz = '0.08 -0.08475 -0.0389' rpy = '0 0 0'/>
-        <parent link = '${prefix}chassis_link'/>
-        <child link = '${prefix}front_right_wheel_link'/>
+        <parent link = '${prefix}_chassis_link'/>
+        <child link = '${prefix}_front_right_wheel_link'/>
         <axis xyz = '0 1 0' rpy = '0 0 0'/>
         <dynamics damping = '${d}'/>
     </joint>
     <!-- front left wheel link -->
-    <link name = '${prefix}front_left_wheel_link'>
+    <link name = '${prefix}_front_left_wheel_link'>
         <visual>
             <origin xyz = '0 0 0' rpy = '1.570796 0 0'/>
@@ -130,13 +130,13 @@
     </link>
     <!-- front left wheel to chassis joint -->
-    <joint name = '${prefix}front_left_joint' type = 'continuous'>
+    <joint name = '${prefix}_front_left_joint' type = 'continuous'>
         <origin xyz = '0.08 0.08475 -0.0389' rpy = '0 0 0'/>
-        <parent link = '${prefix}chassis_link'/>
-        <child link = '${prefix}front_left_wheel_link'/>
+        <parent link = '${prefix}_chassis_link'/>
+        <child link = '${prefix}_front_left_wheel_link'/>
         <axis xyz = '0 1 0' rpy = '0 0 0'/>
         <dynamics damping = '${d}'/>
     </joint>
     <!-- back right wheel link -->
-    <link name = '${prefix}back_right_wheel_link'>
+    <link name = '${prefix}_back_right_wheel_link'>
         <visual>
             <origin xyz = '0 0 0' rpy = '1.570796 0 0'/>
@@ -162,13 +162,13 @@
     </link>
     <!-- back right wheel to chassis joint -->
-    <joint name = '${prefix}back_right_joint' type = 'continuous'>
+    <joint name = '${prefix}_back_right_joint' type = 'continuous'>
         <origin xyz = '-0.08 -0.08475 -0.0389' rpy = '0 0 0'/>   <!-- z was -0.03946 -->
-        <parent link = '${prefix}chassis_link'/>
-        <child link = '${prefix}back_right_wheel_link'/>
+        <parent link = '${prefix}_chassis_link'/>
+        <child link = '${prefix}_back_right_wheel_link'/>
         <axis xyz = '0 1 0' rpy = '0 0 0'/>
         <dynamics damping = '${d}'/>
     </joint>
     <!-- back left wheel link -->
-    <link name = '${prefix}back_left_wheel_link'>
+    <link name = '${prefix}_back_left_wheel_link'>
         <visual>
             <origin xyz = '0 0 0' rpy = '1.570796 0 0'/>
@@ -194,8 +194,8 @@
     </link>
     <!-- back left wheel to chassis joint -->
-    <joint name = '${prefix}back_left_joint' type = 'continuous'>
+    <joint name = '${prefix}_back_left_joint' type = 'continuous'>
         <origin xyz = '-0.08 0.08475 -0.0389' rpy = '0 0 0'/> <!-- z was -0.03954 -->
-        <parent link = '${prefix}chassis_link'/>
-        <child link = '${prefix}back_left_wheel_link'/>
+        <parent link = '${prefix}_chassis_link'/>
+        <child link = '${prefix}_back_left_wheel_link'/>
         <axis xyz = '0 1 0' rpy = '0 0 0'/>
         <dynamics damping = '${d}'/>

File: mrs_robot_launcher/urdf/X3/robot_peripherals.xacro (robot description, xacro)
@@ -3,5 +3,5 @@
     <!--            PERIPHERALS & JOINTS             -->
     <!-- lidar link -->
-    <link name = '${prefix}lidar_link'>
+    <link name = '${prefix}_lidar_link'>
         <visual>
             <origin xyz = '0 0 0' rpy = '1.570796 0 1.570796'/>
@@ -27,11 +27,11 @@
     </link>
     <!-- lidar to chassis joint -->
-    <joint name = '${prefix}lidar_joint' type = 'fixed'>
+    <joint name = '${prefix}_lidar_joint' type = 'fixed'>
         <origin xyz = '0.0405 5.25826986680105E-05 0.08285' rpy = '0 0 0'/>
-        <parent link = '${prefix}chassis_link'/>
-        <child link = '${prefix}lidar_link'/>
+        <parent link = '${prefix}_chassis_link'/>
+        <child link = '${prefix}_lidar_link'/>
     </joint>
     <!-- camera link -->
-    <link name = '${prefix}camera_link'>
+    <link name = '${prefix}_camera_link'>
         <visual>
             <origin xyz = '0 0 0' rpy = '0 0 0'/>
@@ -52,17 +52,17 @@
     </link>
     <!-- camera to chassis joint -->
-    <joint name = '${prefix}camera_joint' type = 'fixed'>
+    <joint name = '${prefix}_camera_joint' type = 'fixed'>
         <origin xyz = '0.057105 1.7948E-05 0.03755' rpy = '0 0 0'/>
-        <parent link = '${prefix}chassis_link'/>
-        <child link = '${prefix}camera_link'/>
+        <parent link = '${prefix}_chassis_link'/>
+        <child link = '${prefix}_camera_link'/>
     </joint>
     <!-- optical link for camera coordinate frame -->
-    <link name = '${prefix}camera_link_optical'>
+    <link name = '${prefix}_camera_link_optical'>
     </link>
     <!-- optical camera link to actual camera link joint: -->
-    <joint name = '${prefix}camera_optical_joint' type = 'fixed'>
+    <joint name = '${prefix}_camera_optical_joint' type = 'fixed'>
         <origin xyz = '0 0 0' rpy = '-1.570796 0 -1.570796'/>
-        <parent link = '${prefix}camera_link'/>
-        <child link = '${prefix}camera_link_optical'/>
+        <parent link = '${prefix}_camera_link'/>
+        <child link = '${prefix}_camera_link_optical'/>
     </joint>
 </robot>

Commit message: accurate RVIZ colours

File: mrs_robot_launcher/urdf/X3/robot_body.xacro (robot description, xacro)
@@ -10,6 +10,9 @@
         <color rgba = '0.1 0.1 0.1 1'/>
     </material>
-    <material name = 'green'>
-        <color rgba = '0 0.7 0 1'/>
+    <material name = 'red'>
+        <color rgba = '1 0 0 1'/>
+    </material>
+    <material name = 'blue'>
+        <color rgba = '0 0 1 1'/>
     </material>
     <material name = 'gray'>
@@ -48,5 +51,10 @@
                 <mesh filename = 'file://$(find mrs_robot_launcher)/meshes/chassis.STL'/>
             </geometry>
-            <material name = 'green'/>
+            <xacro:if value = "${capability == 'depth'}">
+                <material name = 'blue'/>
+            </xacro:if>
+            <xacro:if value = "${capability == 'thermal'}">
+                <material name = 'red'/>
+            </xacro:if>
         </visual>
         <collision>
