Commit message: added a parameter to control the effort of each of the joints. however, it is worth noting that, as per https://wiki.ros.org/urdf/XML/joint, continuous joints do not need a limit tag

File: mrs_robot_launcher/urdf/agent_body.xacro (robot description, xacro)
@@ -4,4 +4,5 @@
     <xacro:property name = "a" value = "1.0"/>          <!-- scalar used for inertia-->
     <xacro:property name = "d" value = "1.0"/>          <!-- scalar used for damping -->
+    <xacro:property name = "effort" value = "0.5"/>     <!-- scalar used for wheel effort -->
     <xacro:property name = "o" value = "0.0"/>          <!-- tuneable offset for wheel collision -->
     <xacro:property name = "c_mass" value = "2.415"/>   <!-- chassis mass in kg -->
@@ -113,5 +114,5 @@
         <axis xyz = "0 1 0" rpy = "0 0 0"/>
         <dynamics damping = "${d}"/>
-        <limit effort = "0.05" velocity = "10.0"/>
+        <limit effort = "${effort}" velocity = "10.0"/>
     </joint>
     <!-- front left wheel link -->
@@ -147,5 +148,5 @@
         <axis xyz = "0 1 0" rpy = "0 0 0"/>
         <dynamics damping = "${d}"/>
-        <limit effort = "0.05" velocity = "10.0"/>
+        <limit effort = "${effort}" velocity = "10.0"/>
     </joint>
     <!-- back right wheel link -->
@@ -181,5 +182,5 @@
         <axis xyz = "0 1 0" rpy = "0 0 0"/>
         <dynamics damping = "${d}"/>
-        <limit effort = "0.05" velocity = "10.0"/>
+        <limit effort = "${effort}" velocity = "10.0"/>
     </joint>
     <!-- back left wheel link -->
@@ -215,5 +216,5 @@
         <axis xyz = "0 1 0" rpy = "0 0 0"/>
         <dynamics damping = "${d}"/>
-        <limit effort = "0.05" velocity = "10.0"/>
+        <limit effort = "${effort}" velocity = "10.0"/>
     </joint>
 </robot>
