Commit message: modify URDF to work in Gazebo

File: mrs_robot_launcher/urdf/goal/goal.urdf.xacro (robot description, xacro)
@@ -3,7 +3,10 @@
     <!-- ARGUMENTS AND PARAMETERS -->
     <xacro:arg name = "goal_name" default = "goal"/>
+    <xacro:arg name = "goal_type" default = "typeA"/>
     <xacro:property name = "prefix" value = "$(arg goal_name)"/>
+    <xacro:property name = "type" value = "$(arg goal_type)"/>
     <!-- DEBUG MESSAGES -->
     <DEBUG_MSG value = "Loading prefix with value ${prefix}"/>
+    <DEBUG_MSG value = "Loading type with value ${type}"/>
     <!-- INCLUDE FILES -->
     <xacro:include filename = "goal_body.xacro"/>

File: mrs_robot_launcher/urdf/goal/goal_body.xacro (robot description, xacro)
@@ -1,11 +1,28 @@
 <?xml version = "1.0"?>
 <robot xmlns:xacro = "http://www.ros.org/wiki/xacro">
+    <!-- PROPERTIES -->
+    <xacro:property name = "a" value = "1.0"/>          <!-- scalar used for inertia-->
     <!-- MATERIALS -->
-    <material name = "green">
-        <color rgba = "0 1 0 0.5"/>
+    <material name = "blue">
+        <color rgba = "0.18 0.61 0.95 0.9"/>
     </material>
+    <material name = "red">
+        <color rgba = "0.95 0.18 0.18 0.9"/>
+    </material>
+    <!-- MACROS -->
+    <xacro:macro name = "cylinder_inertia" params = "mass radius length">
+        <inertia
+            ixx = "${a * mass * (3 * radius**2 + length**2) / 12}"
+            ixy = "0"
+            ixz = "0"
+            iyy = "${a * mass * (3 * radius**2 + length**2) / 12}"
+            iyz = "0"
+            izz = "${a * mass * radius**2 / 12}"
+        />
+    </xacro:macro>
     <!-- LINKS -->
     <!-- base link -->
-    <link name = "${prefix}_base_link"/>
+    <link name = "${prefix}_base_link">
+    </link>
     <!-- body link -->
     <link name = "${prefix}_body_link">
@@ -15,6 +32,25 @@
                 <cylinder radius = "0.1" length = "0.0095"/>
             </geometry>
-            <material name = "green"/>
+            <xacro:if value = "${type == 'typeA'}">
+                <material name = "blue"/>
+            </xacro:if>
+            <xacro:if value = "${type == 'typeB'}">
+                <material name = "red"/>
+            </xacro:if>
         </visual>
+        <collision>
+            <origin xyz = "0 0 0.00475" rpy = "0 0 0"/>
+            <geometry>
+                <cylinder radius = "0.1" length = "0.0095"/>
+            </geometry>
+        </collision>
+        <inertial>
+            <mass value = "0.01"/>
+            <xacro:cylinder_inertia
+                mass = "0.01"
+                radius = "0.1"
+                length = "0.0095"
+            />
+        </inertial>
     </link>
     <!-- JOINTS -->
