Commit message: fix goal collision - set height of collision cylinder to be super small so that the agent doesn't visibly drive over the goal - added a static tag, so that even small movements or slippage between wheel and collision body are negated

File: mrs_robot_launcher/urdf/goal/goal_body.xacro (robot description, xacro)
@@ -40,7 +40,7 @@
         </visual>
         <collision>
-            <origin xyz = "0 0 0.00475" rpy = "0 0 0"/>
+            <origin xyz = "0 0 0" rpy = "0 0 0"/>
             <geometry>
-                <cylinder radius = "0.1" length = "0.0095"/>
+                <cylinder radius = "0.1" length = "0.0000001"/>
             </geometry>
         </collision>
@@ -54,4 +54,7 @@
         </inertial>
     </link>
+    <gazebo>
+        <static>true</static>
+    </gazebo>
     <!-- JOINTS -->
     <joint name = "${prefix}_base_joint" type = "fixed">
