Commit message: add a ``max_vel`` property, used for setting wheel velocity limits

File: mrs_robot_launcher/urdf/agent/agent_body.xacro (robot description, xacro)
@@ -5,4 +5,5 @@
     <xacro:property name = "d" value = "1.0"/>          <!-- scalar used for damping -->
     <xacro:property name = "effort" value = "0.5"/>     <!-- scalar used for wheel effort -->
+    <xacro:property name = "max_vel" value = "50.0"/>   <!-- scalar used for max wheel velocity -->
     <xacro:property name = "o" value = "0.0"/>          <!-- tuneable offset for wheel collision -->
     <xacro:property name = "c_mass" value = "2.415"/>   <!-- chassis mass in kg -->
@@ -114,5 +115,5 @@
         <axis xyz = "0 1 0" rpy = "0 0 0"/>
         <dynamics damping = "${d}"/>
-        <limit effort = "${effort}" velocity = "10.0"/>
+        <limit effort = "${effort}" velocity = "${max_vel}"/>
     </joint>
     <!-- front left wheel link -->
@@ -148,5 +149,5 @@
         <axis xyz = "0 1 0" rpy = "0 0 0"/>
         <dynamics damping = "${d}"/>
-        <limit effort = "${effort}" velocity = "10.0"/>
+        <limit effort = "${effort}" velocity = "${max_vel}"/>
     </joint>
     <!-- back right wheel link -->
@@ -182,5 +183,5 @@
         <axis xyz = "0 1 0" rpy = "0 0 0"/>
         <dynamics damping = "${d}"/>
-        <limit effort = "${effort}" velocity = "10.0"/>
+        <limit effort = "${effort}" velocity = "${max_vel}"/>
     </joint>
     <!-- back left wheel link -->
@@ -216,5 +217,5 @@
         <axis xyz = "0 1 0" rpy = "0 0 0"/>
         <dynamics damping = "${d}"/>
-        <limit effort = "${effort}" velocity = "10.0"/>
+        <limit effort = "${effort}" velocity = "${max_vel}"/>
     </joint>
 </robot>

Commit message: change xacro property ordering

File: mrs_robot_launcher/urdf/agent/agent_body.xacro (robot description, xacro)
@@ -4,9 +4,9 @@
     <xacro:property name = "a" value = "1.0"/>          <!-- scalar used for inertia-->
     <xacro:property name = "d" value = "1.0"/>          <!-- scalar used for damping -->
-    <xacro:property name = "effort" value = "0.5"/>     <!-- scalar used for wheel effort -->
-    <xacro:property name = "max_vel" value = "50.0"/>   <!-- scalar used for max wheel velocity -->
     <xacro:property name = "o" value = "0.0"/>          <!-- tuneable offset for wheel collision -->
     <xacro:property name = "c_mass" value = "2.415"/>   <!-- chassis mass in kg -->
     <xacro:property name = "w_mass" value = "0.058"/>   <!-- wheel mass in kg -->
+    <xacro:property name = "effort" value = "0.5"/>     <!-- scalar used for wheel effort -->
+    <xacro:property name = "max_vel" value = "50.0"/>   <!-- scalar used for max wheel velocity -->
     <!-- MATERIALS -->
     <material name = "black">
